Commit message: Added UAV with sensor

File: models/rotors_description/urdf/component_snippets.xacro (robot description, xacro)
@@ -32,4 +32,73 @@
     </gazebo>
   </xacro:macro>
+  <xacro:macro name="lidar_macro"
+  params="namespace enable_visual lidar_suffix parent_link *cylinder *origin">
+  <link name="${namespace}/lidar_${lidar_suffix}_link">
+    <collision>
+      <origin xyz="0 0 0" rpy="0 0 0" />
+      <geometry>
+        <xacro:insert_block name="cylinder" />
+      </geometry>
+    </collision>
+    <xacro:if value="${enable_visual}">
+      <visual>
+        <origin xyz="0 0 0" rpy="0 1.57079632679 0" />
+        <geometry>
+          <xacro:insert_block name="cylinder" />
+        </geometry>
+        <material name="red" />
+      </visual>
+    </xacro:if>
+      <inertial>
+        <mass value="1e-5" />
+        <origin xyz="0 0 0" rpy="0 0 0" />
+      <inertia ixx="1e-6" ixy="0" ixz="0" iyy="1e-6" iyz="0" izz="1e-6" />
+    </inertial>
+  </link>
+  <joint name="${namespace}/lidar_${lidar_suffix}_joint" type="fixed">
+    <xacro:insert_block name="origin" />
+    <parent link="${parent_link}" />
+    <child link="${namespace}/lidar_${lidar_suffix}_link" />
+  </joint>
+  <gazebo reference="${namespace}/lidar_${lidar_suffix}_link">
+    <sensor name="${namespace}_lidar_${lidar_suffix}" type="ray">
+      <ray>
+        <scan>
+          <horizontal>
+            <samples>30</samples>
+            <resolution>1</resolution>
+            <min_angle>-0.5236</min_angle>
+            <max_angle>0.5236</max_angle>
+          </horizontal>
+          <vertical>
+            <samples>50</samples>
+            <resolution>1.0</resolution>
+            <min_angle>-0.5236</min_angle>
+            <max_angle>0.5236</max_angle>
+          </vertical>
+        </scan>
+        <range>
+          <min>0.10</min>
+          <max>30.0</max>
+          <resolution>0.01</resolution>
+        </range>
+        <noise>
+          <type>gaussian</type>
+          <mean>0.0</mean>
+          <stddev>0.02</stddev>
+        </noise>
+      </ray>
+      <plugin name="${namespace}_lidar_${lidar_suffix}_controller" filename="libgazebo_ros_laser.so">
+        <robotNamespace>${namespace}</robotNamespace>
+        <rayName>lidar_${lidar_suffix}</rayName>
+        <topicName>laser_scan</topicName>
+        <frameName>lidar_${lidar_suffix}_link</frameName>
+      </plugin>
+      <always_on>1</always_on>
+      <update_rate>20</update_rate>
+      <visualize>true</visualize>
+    </sensor>
+  </gazebo>
+</xacro:macro>
   <!-- Macro to add a camera. -->
   <xacro:macro name="camera_macro"

Commit message: Moved lidar sensor

File: models/rotors_description/urdf/component_snippets.xacro (robot description, xacro)
@@ -68,6 +68,6 @@
             <samples>30</samples>
             <resolution>1</resolution>
-            <min_angle>-0.5236</min_angle>
-            <max_angle>0.5236</max_angle>
+            <min_angle>-3.14</min_angle>
+            <max_angle>3.14</max_angle>
           </horizontal>
           <vertical>

File: models/rotors_description/urdf/iris_sensors_base.xacro (robot description, xacro)
@@ -72,5 +72,5 @@
     >
     <box size="0.05 0.05 0.05" />
-    <origin xyz="0 0 -0.07" rpy="0 0 0"/>
+    <origin xyz="0 0 0.12" rpy="0 0 0"/>
   </xacro:lidar_macro>
   <!-- Instantiate gps plugin. -->
