Commit message: Depth Cam added

File: models/rotors_description/urdf/iris_sensors_base.xacro (robot description, xacro)
@@ -45,5 +45,5 @@
         />
   </xacro:if>
-  <!-- Mount Camera Macro -->
+  <!-- Mount Camera Macro
   <xacro:camera_macro
     namespace="${namespace}"
@@ -63,5 +63,23 @@
     <box size="0.05 0.05 0.05" />
     <origin xyz="0 0 0.07" rpy="0 0 0"/>
-  </xacro:camera_macro>
+  </xacro:camera_macro> -->
+  <xacro:depth_camera_macro
+    namespace="${namespace}"
+    parent_link="base_link"
+    camera_suffix="red_iris"
+    frame_rate="30.0"
+    horizontal_fov="1.3962634"
+    image_width="800"
+    image_height="800"
+    image_format="R8G8B8"
+    min_distance="0.02"
+    max_distance="300"
+    noise_mean="0.0"
+    noise_stddev="0.007"
+    enable_visual="1"
+    >
+    <box size="0.05 0.05 0.05" />
+    <origin xyz="0 0 0.07" rpy="0 0 0"/>
+  </xacro:depth_camera_macro>
   <!-- Mount lidar sensor Macro -->
   <xacro:lidar_macro
